File: kicad/OpenMPW-TR10/OpenMPW-TR10.kicad_sch (KiCad schematic)
At the start: 10 parts, among them J1 Conn_01x11_Pin, J2 Conn_01x11_Pin, J3 Conn_01x11_Pin, J4 Conn_01x11_Pin, J5 Conn_01x02_Pin, U1 TR10

Commit message: Convert  minimum line width 3mil -> 4mil.
Convert  minimum line width 3mil -> 4mil.
Parts:
- U1: footprint OpenMPW-TR10:PAD-44_EP_5x5_Pitch0.2mm -> OpenMPW-TR10:PAD-44_EP_5x5_Pitch0.2032mm
Changed lines of the file:
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@@
 			)
 		)
-		(property "Footprint" "OpenMPW-TR10:PAD-44_EP_5x5_Pitch0.2mm"
+		(property "Footprint" "OpenMPW-TR10:PAD-44_EP_5x5_Pitch0.2032mm"
 			(at 151.384 95.504 0)
 			(effects

Commit message: Support pad pitch 0.12mm.
Support pad pitch 0.12mm.
Parts:
- U1: footprint OpenMPW-TR10:PAD-44_EP_5x5_Pitch0.2032mm -> OpenMPW-TR10:PAD-44_EP_5x5_Pitch0.2216mm
Changed lines of the file:
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@@
 			)
 		)
-		(property "Footprint" "OpenMPW-TR10:PAD-44_EP_5x5_Pitch0.2032mm"
+		(property "Footprint" "OpenMPW-TR10:PAD-44_EP_5x5_Pitch0.2216mm"
 			(at 151.384 95.504 0)
 			(effects
